Commit message: Tried various configuration to stablise the robot

File: src/miniproj/description/crobot.urdf.xacro (robot description, xacro)
@@ -2,3 +2,4 @@
 <robot xmlns:xacro="http://www.ros.org/wiki/xacro" name="crobot">
 	<xacro:include filename="crobot_core.xacro" />
+	<xacro:include filename="crobot_control.xacro" />
 </robot>

File: src/miniproj/description/crobot_core.xacro (robot description, xacro)
@@ -31,8 +31,11 @@
 			</geometry>
 		</collision>
-		<xacro:inertial_box mass="0.5" x="0.3" y="0.3" z="0.15">
+		<xacro:inertial_box mass="1" x="0.3" y="0.3" z="0.15">
 			<origin xyz="0.15 0 0.075" rpy="0 0 0" />
 		</xacro:inertial_box>
 	</link>
+	<gazebo reference="chasis">
+		<material>Gazebo/White</material>
+	</gazebo>
 	<joint name="left_wheel_joint" type="continuous">
 		<parent link="base_link" />
@@ -57,4 +60,9 @@
 		</xacro:inertial_cylinder>
 	</link>
+	<gazebo reference="left_wheel">
+		<material>Gazebo/Orange</material>
+		<!-- <mu>100</mu>
+		<mu2>50</mu2> -->
+	</gazebo>
 	<joint name="right_wheel_joint" type="continuous">
 		<parent link="base_link" />
@@ -79,4 +87,9 @@
 		</xacro:inertial_cylinder>
 	</link>
+	<gazebo reference="right_wheel">
+		<material>Gazebo/Orange</material>
+		<!-- <mu>100</mu>
+		<mu2>50</mu2> -->
+	</gazebo>
 	<joint name="caster_wheel_joint" type="fixed">
 		<parent link="chassis" />
@@ -96,12 +109,17 @@
 			</geometry>
 		</collision>
-		<xacro:inertial_sphere mass="0.1" radius="0.05">
+		<xacro:inertial_sphere mass="0.2" radius="0.05">
 			<origin xyz="0 0 0" rpy="0 0 0" />
 		</xacro:inertial_sphere>
 	</link>
+	<gazebo reference="caster_wheel">
+		<material>Gazebo/Blue</material>
+		<mu>0.001</mu>
+		<mu2>0.001</mu2>
+	</gazebo>
 	<joint name="topbody_joint" type="fixed">
 		<parent link="base_link" />
 		<child link="topbody" />
-		<origin xyz="0 0 0.15" />
+		<origin xyz="0.1 0 0.15" />
 	</joint>
 	<link name="topbody">
@@ -109,5 +127,5 @@
 			<origin xyz="0 0 0.15" />
 			<geometry>
-				<box size="0.1 0.1 0.5" />
+				<box size="0.05 0.05 0.5" />
 			</geometry>
 			<material name="white" />
@@ -116,10 +134,13 @@
 			<origin xyz="0 0 0.15" />
 			<geometry>
-				<box size="0.1 0.1 0.5" />
+				<box size="0.05 0.05 0.5" />
 			</geometry>
 		</collision>
-		<xacro:inertial_box mass="0.1" x="0.1" y="0.1" z="0.5">
+		<xacro:inertial_box mass="0.05" x="0.05" y="0.05" z="0.5">
 			<origin xyz="0 0 0.15" rpy="0 0 0" />
 		</xacro:inertial_box>
 	</link>
+	<gazebo reference="topbody">
+		<material>Gazebo/Gray</material>
+	</gazebo>
 </robot>

Commit message: Added camera plugin and realigned crobot

File: src/miniproj/description/crobot.urdf.xacro (robot description, xacro)
@@ -3,3 +3,4 @@
 	<xacro:include filename="crobot_core.xacro" />
 	<xacro:include filename="crobot_control.xacro" />
+	<xacro:include filename="crobot_camera.xacro" />
 </robot>

File: src/miniproj/description/crobot_control.xacro (robot description, xacro)
@@ -4,4 +4,5 @@
         <plugin name="differential_drive_controller" filename="libgazebo_ros_diff_drive.so">
             <commandTopic>cmd_vel</commandTopic>
+            <odometryTopic>odom</odometryTopic>
             <odometryFrame>odom</odometryFrame>
             <robotBaseFrame>base_link</robotBaseFrame>
@@ -9,5 +10,5 @@
             <wheelDiameter>0.1</wheelDiameter>
             <wheelTorque>200</wheelTorque>
-            <!-- <wheelAcceleration>10</wheelAcceleration> -->
+            <wheelAcceleration>10.0</wheelAcceleration>
             <leftJoint>left_wheel_joint</leftJoint>
             <rightJoint>right_wheel_joint</rightJoint>
@@ -16,4 +17,7 @@
             <publishWheelTF>true</publishWheelTF>
             <publishWheelJointState>true</publishWheelJointState>
+            <publishTf>true</publishTf>
+            <!-- <odometrySource>1</odometrySource> -->
+            <updateRate>100</updateRate>
         </plugin>
     </gazebo>

File: src/miniproj/description/crobot_core.xacro (robot description, xacro)
@@ -8,6 +8,9 @@
 		<color rgba="0 0 0 1" />
 	</material>
+	<material name="red">
+		<color rgba="1 0.3 0.1 1" />
+	</material>
 	<material name="orange">
-		<color rgba="1 0.3 0.1 1" />
+		<color rgba="1 0 0 1" />
 	</material>
 	<link name="base_link"></link>
@@ -144,3 +147,32 @@
 		<material>Gazebo/Gray</material>
 	</gazebo>
+	<joint name="camera_joint" type="fixed">
+		<axis xyz="0 1 0" />
+		<origin xyz="0.17 0 0.45" rpy="0 0 ${pi}" />
+		<parent link="chassis" />
+		<child link="camera_link" />
+	</joint>
+	<link name="camera_link">
+		<collision>
+			<origin xyz="0 0 0" rpy="0 0 0" />
+			<geometry>
+				<box size="0.025 0.025 0.025" />
+			</geometry>
+		</collision>
+		<visual>
+			<origin xyz="0 0 0" rpy="0 0 0" />
+			<geometry>
+				<box size="0.025 0.025 0.025" />
+			</geometry>
+			<material name="red" />
+		</visual>
+		<inertial>
+			<mass value="1e-5" />
+			<origin xyz="0 0 0" rpy="0 0 0" />
+			<inertia ixx="1e-6" ixy="0" ixz="0" iyy="1e-6" iyz="0" izz="1e-6" />
+		</inertial>
+	</link>
+	<gazebo reference="camera_link">
+		<material>Gazebo/Red</material>
+	</gazebo>
 </robot>
