Commit message: Decreased height of the camera

File: src/miniproj/description/crobot_core.xacro (robot description, xacro)
@@ -149,5 +149,5 @@
 	<joint name="camera_joint" type="fixed">
 		<axis xyz="0 1 0" />
-		<origin xyz="0.17 0 0.45" rpy="0 0 ${pi}" />
+		<origin xyz="0.17 0 0.35" rpy="0 0 ${pi}" />
 		<parent link="chassis" />
 		<child link="camera_link" />

Commit message: Changed the angle of camera

File: src/miniproj/description/crobot_core.xacro (robot description, xacro)
@@ -149,5 +149,5 @@
 	<joint name="camera_joint" type="fixed">
 		<axis xyz="0 1 0" />
-		<origin xyz="0.17 0 0.35" rpy="0 0 ${pi}" />
+		<origin xyz="0.17 0 0.35" rpy="0 ${pi/6} ${pi}" />
 		<parent link="chassis" />
 		<child link="camera_link" />

Commit message: Changed the camera height and robot traversal speed

File: src/miniproj/description/crobot_core.xacro (robot description, xacro)
@@ -149,5 +149,5 @@
 	<joint name="camera_joint" type="fixed">
 		<axis xyz="0 1 0" />
-		<origin xyz="0.17 0 0.35" rpy="0 ${pi/6} ${pi}" />
+		<origin xyz="0.17 0 0.5" rpy="0 ${pi/5} ${pi}" />
 		<parent link="chassis" />
 		<child link="camera_link" />
